Commit message: Integrate live sensors and document workspace

File: src/my_robot_description/urdf/my_robot.urdf (robot description, URDF)
Before this commit: robot my_robot, 20 links, 19 joints
Links:
- removed link rplidar_link
- added link laser, mass 0.19; collision cylinder length=0.040 radius=0.035; visual cylinder length=0.040 radius=0.035
Joints:
- joint rplidar_joint: child rplidar_link -> laser

Commit message: Add Arduino MDDS10 motor interface

File: src/my_robot_description/urdf/my_robot.urdf (robot description, URDF)
Before this commit: robot my_robot, 20 links, 19 joints
Links:
- removed link l298n_link
- added link mdds10_link, mass 0.03; collision box size=0.106 0.084 0.024; visual box size=0.106 0.084 0.024
Joints:
- removed joint l298n_joint
- added joint mdds10_joint: type fixed, parent plate_3, child mdds10_link, origin xyz=-0.02 -0.03 0.011 rpy=0 0 0

Commit message: test from laptop:

File: src/my_robot_description/urdf/my_robot.urdf (robot description, URDF)
Before this commit: robot my_robot, 20 links, 19 joints
Links:
- removed link mdds10_link
- added link l298n_link, mass 0.03; collision box size=0.106 0.084 0.024; visual box size=0.106 0.084 0.024
Joints:
- removed joint mdds10_joint
- added joint l298n_joint: type fixed, parent plate_3, child l298n_link, origin xyz=-0.02 -0.03 0.011 rpy=0 0 0
